Commit message: initial commit

File: robots/igus_lineaJoint_SV.urdf.xacro (robot description, xacro)
@@ -45,3 +45,221 @@
     <dynamics damping="1000.0"/>
   </joint>
+  <link name="link1">
+    <visual>
+    <origin rpy="0 0 0" xyz="0 0 0"/>
+      <geometry>
+          <mesh filename="package://cpr_robot/robots/igus_5DOF_SV/Joint1.dae"  scale="0.001 0.001 0.001"/>
+        </geometry>
+    </visual>
+    <collision>
+      <origin xyz="0 0 0" rpy="0 0 0" />
+      <geometry>
+          <mesh filename="package://cpr_robot/robots/igus_5DOF_SV/Joint1Coll.dae" scale="0.001 0.001 0.001"/>
+        </geometry>
+    </collision>
+  </link>
+  <link name="link2">
+    <visual>
+    <origin rpy="0 0 0" xyz="0 0 0"/>
+      <geometry>
+          <mesh filename="package://cpr_robot/robots/igus_5DOF_SV/Joint2.dae"  scale="0.001 0.001 0.001"/>
+        </geometry>
+    </visual>
+    <collision>
+      <origin xyz="0 0 0" rpy="0 0 0" />
+      <geometry>
+          <mesh filename="package://cpr_robot/robots/igus_5DOF_SV/Joint2Coll.dae" scale="0.001 0.001 0.001"/>
+        </geometry>
+    </collision>
+  </link>
+  <link name="link3">
+    <visual>
+    <origin rpy="0 0 0" xyz="0 0 0"/>
+      <geometry>
+          <mesh filename="package://cpr_robot/robots/igus_5DOF_SV/Joint3.dae"  scale="0.001 0.001 0.001"/>
+        </geometry>
+    </visual>
+    <collision>
+      <origin xyz="0 0 0" rpy="0 0 0" />
+      <geometry>
+          <mesh filename="package://cpr_robot/robots/igus_5DOF_SV/Joint3Coll.dae" scale="0.001 0.001 0.001"/>
+        </geometry>
+    </collision>
+  </link>
+  <link name="link4">
+    <visual>
+    <origin rpy="0 0 0" xyz="0 0 0"/>
+      <geometry>
+          <mesh filename="package://cpr_robot/robots/igus_5DOF_SV/Joint4.dae"  scale="0.001 0.001 0.001"/>
+        </geometry>
+    </visual>
+    <collision>
+      <origin xyz="0 0 0" rpy="0 0 0" />
+      <geometry>
+          <mesh filename="package://cpr_robot/robots/igus_5DOF_SV/Joint4Coll.dae" scale="0.001 0.001 0.001"/>
+        </geometry>
+    </collision>
+  </link>
+  <link name="link5">
+    <visual>
+    <origin rpy="0 0 0" xyz="0 0 -0.0045"/>
+      <geometry>
+          <mesh filename="package://cpr_robot/robots/igus_5DOF_SV/Joint5.dae"  scale="0.001 0.001 0.001"/>
+        </geometry>
+    </visual>
+    <collision>
+      <origin xyz="0 0 0" rpy="0 0 -0.0045" />
+      <geometry>
+          <mesh filename="package://cpr_robot/robots/igus_5DOF_SV/Joint5Coll.dae" scale="0.001 0.001 0.001"/>
+        </geometry>
+    </collision>
+  </link>
+  <joint name="joint1" type="continuous">
+    <axis xyz="0 0 1"/>
+    <parent link="igus_base_link"/>
+    <child link="link1"/>
+    <origin rpy="0 0 0" xyz="0 0 0.1275"/>
+    <limit effort="100" velocity="30"/>
+    <joint_properties damping="0.0" friction="0.0"/>
+  </joint>
+ <joint name="joint2" type="continuous">
+    <axis xyz="0 1 0"/>
+    <parent link="link1"/>
+    <child link="link2"/>
+    <origin rpy="0 0 0" xyz="0 0 0.10025"/>
+    <limit effort="100" velocity="30"/>
+    <joint_properties damping="0.0" friction="0.0"/>
+  </joint>
+ <joint name="joint3" type="continuous">
+    <axis xyz="0 1 0"/>
+    <parent link="link2"/>
+    <child link="link3"/>
+    <origin rpy="0 1.57079632679 0" xyz="0 0 0.270"/>
+    <limit effort="100" velocity="30"/>
+    <joint_properties damping="0.0" friction="0.0"/>
+  </joint>
+ <joint name="joint4" type="continuous">
+    <axis xyz="0 1 0"/>
+    <parent link="link3"/>
+    <child link="link4"/>
+    <origin rpy="0 0 0" xyz="0 0 0.240"/>
+    <limit effort="100" velocity="30"/>
+    <joint_properties damping="0.0" friction="0.0"/>
+  </joint>
+ <joint name="joint5" type="continuous">
+    <axis xyz="0 0 1"/>
+    <parent link="link4"/>
+    <child link="link5"/>
+    <origin rpy="0 0 0" xyz="0 0 0.1835"/>
+    <limit effort="100" velocity="30"/>
+    <joint_properties damping="0.0" friction="0.0"/>
+  </joint>
+  <transmission name="tran_prismatic">
+    <type>transmission_interface/SimpleTransmission</type>
+    <joint name="arm_joint">
+      <hardwareInterface>hardware_interface/PositionJointInterface</hardwareInterface>
+    </joint>
+    <actuator name="tran_prismatic_motor">
+      <mechanicalReduction>1</mechanicalReduction>
+    </actuator>
+  </transmission>
+  <transmission name="tran_roll">
+    <type>transmission_interface/SimpleTransmission</type>
+    <joint name="joint1">
+      <hardwareInterface>hardware_interface/PositionJointInterface</hardwareInterface>
+    </joint>
+    <actuator name="tran_roll_motor">
+      <mechanicalReduction>1</mechanicalReduction>
+    </actuator>
+  </transmission>
+  <transmission name="tran_1">
+    <type>transmission_interface/SimpleTransmission</type>
+    <joint name="joint2">
+      <hardwareInterface>hardware_interface/PositionJointInterface</hardwareInterface>
+    </joint>
+    <actuator name="tran_1_motor">
+      <mechanicalReduction>1</mechanicalReduction>
+    </actuator>
+  </transmission>
+   <transmission name="tran_2">
+    <type>transmission_interface/SimpleTransmission</type>
+    <joint name="joint3">
+      <hardwareInterface>hardware_interface/PositionJointInterface</hardwareInterface>
+    </joint>
+    <actuator name="tran_2_motor">
+      <mechanicalReduction>1</mechanicalReduction>
+    </actuator>
+  </transmission>
+   <transmission name="tran_3">
+    <type>transmission_interface/SimpleTransmission</type>
+    <joint name="joint4">
+      <hardwareInterface>hardware_interface/PositionJointInterface</hardwareInterface>
+    </joint>
+    <actuator name="tran_3_motor">
+      <mechanicalReduction>1</mechanicalReduction>
+    </actuator>
+  </transmission>
+   <transmission name="tran_4">
+    <type>transmission_interface/SimpleTransmission</type>
+    <joint name="joint5">
+      <hardwareInterface>hardware_interface/PositionJointInterface</hardwareInterface>
+    </joint>
+    <actuator name="tran_4_motor">
+      <mechanicalReduction>1</mechanicalReduction>
+    </actuator>
+  </transmission>
+    <gazebo reference="linear_link">
+            <material>Gazebo/Grey</material>
+            <kp>1000000</kp>
+            <kd>1000000</kd>
+            <mu1>500</mu1>
+            <mu2>200</mu2>
+        </gazebo>
+    <gazebo reference="igus_base_link">
+            <material>Gazebo/Grey</material>
+            <kp>1000000</kp>
+            <kd>1000000</kd>
+            <mu1>1</mu1>
+            <mu2>1</mu2>
+        </gazebo>
+        <!-- Link1 -->
+        <gazebo reference="link1">
+            <material>Gazebo/White</material>
+            <kp>1000000</kp>
+            <kd>1000000</kd>
+            <mu1>0.2</mu1>
+            <mu2>0.2</mu2>
+        </gazebo>
+        <!-- Link2 -->
+        <gazebo reference="link2">
+            <material>Gazebo/White</material>
+            <kp>1000000</kp>
+            <kd>1000000</kd>
+            <mu1>0.2</mu1>
+            <mu2>0.2</mu2>
+        </gazebo>
+        <!-- Link3 -->
+        <gazebo reference="link3">
+            <material>Gazebo/White</material>
+           <kp>1000000</kp>
+            <kd>1000000</kd>
+            <mu1>0.2</mu1>
+            <mu2>0.2</mu2>
+        </gazebo>
+        <!-- Link4 -->
+        <gazebo reference="link4">
+            <material>Gazebo/White</material>
+            <kp>1000000</kp>
+            <kd>1000000</kd>
+            <mu1>0.2</mu1>
+            <mu2>0.2</mu2>
+        </gazebo>
+        <!-- Link5 -->
+        <gazebo reference="link5">
+            <material>Gazebo/White</material>
+            <kp>1000000</kp>
+            <kd>1000000</kd>
+            <mu1>0.2</mu1>
+            <mu2>0.2</mu2>
+        </gazebo>
 </robot>
